Commit message: PR feedback

File: resources/urdf/hsrb.urdf (robot description, URDF)
Before this commit: robot hsrb, 49 links, 48 joints
Joints:
- joint base_b_bumper_joint: type revolute -> fixed
- joint base_f_bumper_joint: type revolute -> fixed
- joint wrist_ft_sensor_frame_joint: type revolute -> fixed
